File: PTP_Ivan_Brajkovic_Project1AAA.kicad_sch (KiCad schematic)
At the start: 45 parts, among them J1 Screw_Terminal_01x02, SW1 SW_Push_Dual_x2, SW2 SW2, U1 LM2574N-5, U2 4027, U3 4027, U4 74LS47, U5 FYS-3911BUHR-21, U6 74LVC1G11, U7 NE555P

Commit message: lv5
Parts:
- D2, D3, D5: footprint (none) -> LED_THT:LED_D5.0mm
- U6: footprint SOT-23-6:SOT-23-6 -> Package_TO_SOT_SMD:SOT-23-6
Other:
- note added: "555 timer"
- note added: "JK bistabil"
- note added: "LED diode"
- note added: "Montažne rupe"
- note added: "Napajanje"
- note added: "Napajanje bistabila"
- note added: "Reset brojača"
- note added: "Tipkalo i ulaz radnog takta"
Changed lines of the file:
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@@
 		(comment 1 "izradio: Ivan Brajković")
 	)
+	(text "Montažne rupe"
+		(exclude_from_sim no)
+		(at 179.324 131.572 0)
+		(effects
+			(font
+				(size 1.27 1.27)
+			)
+		)
+	)
+	(text "Tipkalo i ulaz radnog takta"
+		(exclude_from_sim no)
+		(at 28.956 73.152 0)
+		(effects
+			(font
+				(size 1.27 1.27)
+			)
+		)
+	)
+	(text "Napajanje bistabila"
+		(exclude_from_sim no)
+		(at 129.032 17.78 0)
+		(effects
+			(font
+				(size 1.27 1.27)
+			)
+		)
+	)
+	(text "LED diode"
+		(exclude_from_sim no)
+		(at 192.532 17.78 0)
+		(effects
+			(font
+				(size 1.27 1.27)
+			)
+		)
+	)
+	(text "Reset brojača"
+		(exclude_from_sim no)
+		(at 117.094 131.318 0)
+		(effects
+			(font
+				(size 1.27 1.27)
+			)
+		)
+	)
+	(text "JK bistabil"
+		(exclude_from_sim no)
+		(at 90.932 71.374 0)
+		(effects
+			(font
+				(size 1.27 1.27)
+			)
+		)
+	)
+	(text "Napajanje"
+		(exclude_from_sim no)
+		(at 23.114 17.018 0)
+		(effects
+			(font
+				(size 1.27 1.27)
+			)
+		)
+	)
+	(text "555 timer"
+		(exclude_from_sim no)
+		(at 20.574 132.08 0)
+		(effects
+			(font
+				(size 1.27 1.27)
+			)
+		)
+	)
 	(junction
 		(at 33.02 33.02)
@@
 		)
 	)
+	(polyline
+		(pts
+			(xy 106.68 198.12) (xy 109.22 198.12)
+		)
+		(stroke
+			(width 0)
+			(type default)
+		)
+	)
 	(wire
 		(pts
@@
 		)
 	)
+	(polyline
+		(pts
+			(xy 115.57 12.7) (xy 115.57 67.31)
+		)
+		(stroke
+			(width 0)
+			(type dash_dot)
+		)
+	)
 	(wire
 		(pts
@@
 		)
 	)
+	(polyline
+		(pts
+			(xy 167.64 127) (xy 167.64 198.12)
+		)
+		(stroke
+			(width 0)
+			(type dash_dot)
+		)
+	)
 	(wire
 		(pts
@@
 		)
 	)
+	(polyline
+		(pts
+			(xy 11.43 127) (xy 285.75 127)
+		)
+		(stroke
+			(width 0)
+			(type dash_dot)
+		)
+	)
 	(wire
 		(pts
@@
 		)
 	)
+	(polyline
+		(pts
+			(xy 194.31 67.31) (xy 194.31 127)
+		)
+		(stroke
+			(width 0)
+			(type dash_dot)
+		)
+	)
 	(wire
 		(pts
@@
 		)
 	)
+	(polyline
+		(pts
+			(xy 80.01 67.31) (xy 80.01 127)
+		)
+		(stroke
+			(width 0)
+			(type dash_dot)
+		)
+	)
 	(wire
 		(pts
@@
 		)
 	)
+	(polyline
+		(pts
+			(xy 12.7 67.31) (xy 285.75 67.31)
+		)
+		(stroke
+			(width 0)
+			(type dash_dot)
+		)
+	)
+	(polyline
+		(pts
+			(xy 181.61 11.43) (xy 181.61 67.31)
+		)
+		(stroke
+			(width 0)
+			(type dash_dot)
+		)
+	)
 	(wire
 		(pts
@@
 		)
 	)
+	(polyline
+		(pts
+			(xy 106.68 127) (xy 106.68 198.12)
+		)
+		(stroke
+			(width 0)
+			(type dash_dot)
+		)
+	)
 	(wire
 		(pts
@@
 			)
 		)
-		(property "Footprint" ""
+		(property "Footprint" "LED_THT:LED_D5.0mm"
 			(at 227.33 52.07 0)
 			(effects
@@
 			)
 		)
-		(property "Footprint" "SOT-23-6:SOT-23-6"
+		(property "Footprint" "Package_TO_SOT_SMD:SOT-23-6"
 			(at 147.32 148.59 0)
 			(effects
@@
 			)
 		)
-		(property "Footprint" ""
+		(property "Footprint" "LED_THT:LED_D5.0mm"
 			(at 227.33 39.37 0)
 			(effects
@@
 			)
 		)
-		(property "Footprint" ""
+		(property "Footprint" "LED_THT:LED_D5.0mm"
 			(at 227.33 45.72 0)
 			(effects
@@
 		)
 		(property "Value" "+5V"
-			(at 196.85 93.98 0)
+			(at 199.39 97.7899 0)
 			(effects
 				(font
 					(size 1.27 1.27)
 				)
+				(justify left)
 			)
 		)
